File: PCBs/displays.sch (KiCad schematic (older format))
At the start: 46 parts, among them U2 HT1632C-52LQFP, U3 HT1632C-52LQFP

Commit message: Rerouted scratchpad and added to main schematic
Rerouted the scratchpad traces so that it has only 9 common pins, and two sets of anodes 
A-H and A-P for 16 segment, where each common goes to half a 16 seg digit, and 7 segments respectively, where each common goes to two 7 seg digits. I plan to tie the first set of A-H together with the second A-H, but the option to separately multiplex them is there.
Also replaced the 1mm pitch headers with 2.54mm headers
Added a symbol to the library and added it to the main UFC schematic.
Parts:
- removed DS1: 14Segx2ChromeLED, UFC:SDDCN40G2W, symbol UFClib:14Segx2ChromeLED
- removed DS2: 7Segx3ChromeLED, UFC:SDTC39G2W, symbol UFClib:7Segx3ChromeLED
- removed DS3: 7Segx4ChromeLED, UFC:SDQC39G2W, symbol UFClib:7Segx4ChromeLED
- added DS1: Scratchpad, symbol UFClib:Scratchpad
- renumbered DS4 to DS2, DS5 to DS3, DS6 to DS4, DS7 to DS5, DS8 to DS6, DS14 to DS7, DS15 to DS8
Connections:
- wire segments 315 -> 291
Other:
- note added: "DIG0-3 controls the halves of the two 16 segment digits\nDIG4-8 controls the 7 segment digits, 2 digits per common pin"
- moved on the sheet: DS7, DS8
